File: smd-balanced.kicad_pcb (KiCad board)
At the start: 2 copper layers, 92.5 x 50 mm, 54 parts, among them J1 Conn_01x01_Female, J10 Conn_01x01_Female, J11 Conn_01x01_Female, J2 Conn_01x01_Female, J3 Conn_01x01_Female, J4 Conn_01x01_Female, J6 Conn_01x01_Female, J7 Conn_01x01_Female, J8 Conn_01x01_Female, J9 Conn_01x01_Female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

Commit message: Add files via upload
Parts:
- removed REF**: OSHW-Logo_19x20mm_SilkScreen, Symbol:OSHW-Logo_19x20mm_SilkScreen
- removed U2: NE5534PS, Package_SO:PowerIntegrations_SO-8
- D1: value BZT52C18-7-F -> MMSZ11T1G
- U1: value NE5534PS -> TL082CDE4; footprint Package_SO:PowerIntegrations_SO-8 -> Package_SO:SOIC-8_3.9x4.9mm_P1.27mm
- moved U1 22.5 mm to (85.8, 58.8)
- moved R13 21.0 mm to (74.0, 45.5)
- moved R14 21.0 mm to (74.0, 48.0)
- moved R15 21.0 mm to (74.0, 50.5)
- moved R16 21.0 mm to (74.0, 53.0)
- moved R17 21.0 mm to (74.5, 55.5)
- moved R2 21.0 mm to (73.8, 43.0)
- moved SW1 21.0 mm to (67.1, 50.6)
- moved SW2 9.62 mm to (67.1, 70.1)
- moved R19 9.62 mm to (74.0, 62.5)
- moved R20 9.62 mm to (74.0, 65.0)
- moved R21 9.62 mm to (74.0, 67.5)
- moved R22 9.62 mm to (74.0, 70.0)
- moved R23 9.62 mm to (74.0, 72.5)
- moved R24 9.62 mm to (74.0, 75.0)
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Connections:
- U1 pad 1: Net-(U1-Pad1) -> Rout
- U1 pad 5: Net-(U1-Pad5) -> ind
- U1 pad 6: Rout -> Rin2
- U1 pad 7: VCC -> Rout2
- U1 pad 8: Net-(U1-Pad8) -> VCC
Routing:
- net VCC: track 190.9 -> 102.4 mm
- net ind: track 92.3 -> 65.4 mm, vias 1 -> 3
- net Net-(R18-Pad2): track 3.61 -> 27.4 mm, vias 0 -> 2
- net V-: track 194.0 -> 211.3 mm
- net Rin: track 76.1 -> 63.2 mm, vias 2 -> 0
- net Net-(D2-Pad2): track 66.8 -> 78.0 mm, vias 0 -> 1
- net Rin2: track 58.2 -> 68.9 mm
- net Net-(C8-Pad2): track 11.6 -> 15.8 mm
- net Rout2: track 68.5 -> 71.5 mm
- net Net-(D1-Pad1): track 18.1 -> 20.0 mm
- net Net-(C7-Pad1): track 110.2 -> 111.7 mm
- net /2: track 28.0 -> 29.2 mm, vias 0 -> 1
- net Rout: track 61.6 -> 62.2 mm, vias 0 -> 2
- net Earth: vias 24 -> 21
