File: smd-balanced.sch (KiCad schematic (older format))
At the start: 53 parts, among them J1 Conn_01x01_Female, J10 Conn_01x01_Female, J11 Conn_01x01_Female, J2 Conn_01x01_Female, J3 Conn_01x01_Female, J4 Conn_01x01_Female, J6 Conn_01x01_Female, J7 Conn_01x01_Female, J8 Conn_01x01_Female, J9 Conn_01x01_Female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

Commit message: Add files via upload
Parts:
- removed U1, U2: NE5534PS, Package_SO:PowerIntegrations_SO-8, symbol Amplifier_Operational:NE5534
- added U1: TL082CDE4, Package_SO:SOIC-8_3.9x4.9mm_P1.27mm, symbol Amplifier_Operational:TL082
- D1: value BZT52C18-7-F -> MMSZ11T1G
Connections:
- net GND: now also U1.4 (V-)
- net Rin: now also U1.2 (-)
- net Rin2: now also U1.6 (-)
- net Rout: now also U1.1
- net Rout2: now also U1.7
- net VCC: now also U1.8 (V+)
- net ind: now also U1.5 (+)
- net at D2.2 (A), D3.1 (K), J1.1 (Pin_1)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: now also U1.3 (+)
- no-connect marks 6 -> 0
Changed lines of the file:
@@
 P 6700 1800
 F 0 "D1" V 6654 1880 50  0000 L CNN
-F 1 "BZT52C18-7-F" V 6745 1880 50  0000 L CNN
+F 1 "MMSZ11T1G" V 6745 1880 50  0000 L CNN
 F 2 "Diode_SMD:D_SOD-123" H 6700 1800 50  0001 C CNN
 F 3 "~" H 6700 1800 50  0001 C CNN
@@
 Text GLabel 5050 1000 1    50   Input ~ 0
 VCC
-Text GLabel 5100 2150 1    50   Input ~ 0
+Text GLabel 9100 1000 1    50   Input ~ 0
 VCC
 Wire Wire Line
-	5100 2150 5100 2300
+	9100 1000 9100 1150
 Connection ~ 5050 1050
 Wire Wire Line
@@
 	0    1    1    0
 $EndComp
-NoConn ~ 5200 2300
-NoConn ~ 5200 2900
-NoConn ~ 5300 2900
-Text GLabel 5100 3000 3    50   Input ~ 0
+Text GLabel 9100 1850 3    50   Input ~ 0
 V-
 Wire Wire Line
-	5100 3000 5100 2900
+	9100 1850 9100 1750
 $Comp
 L Device:R R7
@@
 	3750 3350 3750 3600
 Connection ~ 7500 2800
-$Comp
-L Amplifier_Operational:NE5534 U1
-U 1 1 60CCF692
-P 5200 2600
-F 0 "U1" H 5544 2646 50  0000 L CNN
-F 1 "NE5534PS " H 5544 2555 50  0000 L CNN
-F 2 "Package_SO:PowerIntegrations_SO-8" H 5250 2650 50  0001 C CNN
-F 3 "http://www.ti.com/lit/ds/symlink/ne5534.pdf" H 5250 2750 50  0001 C CNN
-	1    5200 2600
-	1    0    0    -1
-$EndComp
 Wire Wire Line
 	7350 2800 7500 2800
@@
 Wire Wire Line
 	5500 2600 5900 2600
-Connection ~ 5500 2600
 $Comp
 L Device:R R9
@@
 Connection ~ 3750 1350
 Connection ~ 8550 3150
-Text GLabel 5850 3600 1    50   Input ~ 0
-VCC
-Wire Wire Line
-	5850 3600 5850 3750
-NoConn ~ 5950 4350
-Text GLabel 5850 4450 3    50   Input ~ 0
-V-
-Wire Wire Line
-	5850 4450 5850 4350
 Wire Wire Line
 	5650 4150 5650 4800
@@
 	6200 4300 6250 4300
 Wire Wire Line
-	6250 4300 6250 4050
-Wire Wire Line
 	6700 2800 6250 2800
-Wire Wire Line
-	6250 2800 6250 4050
-Connection ~ 6250 4050
 Connection ~ 3750 3600
 Wire Wire Line
@@
 Wire Wire Line
 	4800 2700 4900 2700
-$Comp
-L Amplifier_Operational:NE5534 U2
-U 1 1 60D5461E
-P 5950 4050
-F 0 "U2" H 6294 4096 50  0000 L CNN
-F 1 "NE5534PS " H 6294 4005 50  0000 L CNN
-F 2 "Package_SO:PowerIntegrations_SO-8" H 6000 4100 50  0001 C CNN
-F 3 "http://www.ti.com/lit/ds/symlink/ne5534.pdf" H 6000 4200 50  0001 C CNN
-	1    5950 4050
-	1    0    0    -1
-$EndComp
 Text Notes 8800 2800 0    50   ~ 0
 +48 V phantom power
@@
 Wire Wire Line
 	2050 1650 2950 1650
-NoConn ~ 5950 3750
-NoConn ~ 6050 4350
 $Comp
 L Device:D D4
@@
 Wire Wire Line
 	5200 4150 5650 4150
-Connection ~ 5650 4150
 $Comp
 L power:GND #PWR05
@@
 	4600 1350 5050 1350
 Connection ~ 5050 1350
+Wire Wire Line
+	6250 2800 6250 4050
+$Comp
+L Amplifier_Operational:TL082 U1
+U 1 1 60F58229
+P 5200 2600
+F 0 "U1" H 5200 2967 50  0000 C CNN
+F 1 "TL082CDE4" H 5200 2876 50  0000 C CNN
+F 2 "Package_SO:SOIC-8_3.9x4.9mm_P1.27mm" H 5200 2600 50  0001 C CNN
+F 3 "http://www.ti.com/lit/ds/symlink/tl081.pdf" H 5200 2600 50  0001 C CNN
+	1    5200 2600
+	1    0    0    -1
+$EndComp
+Connection ~ 5500 2600
+$Comp
+L Amplifier_Operational:TL082 U1
+U 2 1 60F5B82B
+P 5950 4050
+F 0 "U1" H 5950 4417 50  0000 C CNN
+F 1 "TL082CDE4" H 5950 4326 50  0000 C CNN
+F 2 "Package_SO:SOIC-8_3.9x4.9mm_P1.27mm" H 5950 4050 50  0001 C CNN
+F 3 "http://www.ti.com/lit/ds/symlink/tl081.pdf" H 5950 4050 50  0001 C CNN
+	2    5950 4050
+	1    0    0    -1
+$EndComp
+Connection ~ 6250 4050
+Wire Wire Line
+	6250 4050 6250 4300
+Connection ~ 5650 4150
+$Comp
+L Amplifier_Operational:TL082 U1
+U 3 1 60F654A5
+P 9200 1450
+F 0 "U1" H 9158 1496 50  0000 L CNN
+F 1 "TL082CDE4" H 9158 1405 50  0000 L CNN
+F 2 "Package_SO:SOIC-8_3.9x4.9mm_P1.27mm" H 9200 1450 50  0001 C CNN
+F 3 "http://www.ti.com/lit/ds/symlink/tl081.pdf" H 9200 1450 50  0001 C CNN
+	3    9200 1450
+	1    0    0    -1
+$EndComp
 $EndSCHEMATC

Commit message: Add files via upload
Parts:
- removed U1: TL082CDE4, Package_SO:SOIC-8_3.9x4.9mm_P1.27mm, symbol Amplifier_Operational:TL082
- added C10, C11: 47pF, Capacitor_SMD:C_0201_0603Metric_Pad0.64x0.40mm_HandSolder, symbol Device:C
- added U1: LT6234CS8#PBF, Package_SO:SO-8_3.9x4.9mm_P1.27mm, symbol Amplifier_Operational:LT6234
Connections:
- net GND: now also U1.4 (V-)
- net Rin: now also C10.1, U1.2 (-)
- net Rin2: now also C11.1, U1.6 (-)
- net Rout: now also C10.2, U1.1
- net Rout2: now also C11.2, U1.7
- net VCC: now also U1.8 (V+)
- net ind: now also U1.5 (+)
- net at D2.2 (A), D3.1 (K), J1.1 (Pin_1)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: now also U1.3 (+)
Changed lines of the file:
@@
 Connection ~ 8550 3150
 Wire Wire Line
-	5650 4150 5650 4800
-Wire Wire Line
-	6200 4800 6200 4300
+	5650 4150 5650 4550
+Wire Wire Line
+	6200 4800 6200 4550
 Wire Wire Line
 	6200 4300 6250 4300
@@
 	3850 1050 4600 1050
 Wire Wire Line
-	5500 2600 5500 3400
+	5500 2600 5500 3100
 Wire Wire Line
 	4350 2700 4800 2700
 Wire Wire Line
-	4800 3400 4800 2700
+	4800 3400 4800 3100
 Connection ~ 4800 2700
 Wire Wire Line
@@
 	6250 2800 6250 4050
 $Comp
-L Amplifier_Operational:TL082 U1
-U 1 1 60F58229
+L Amplifier_Operational:LT6234 U1
+U 1 1 610B0893
 P 5200 2600
 F 0 "U1" H 5200 2967 50  0000 C CNN
-F 1 "TL082CDE4" H 5200 2876 50  0000 C CNN
-F 2 "Package_SO:SOIC-8_3.9x4.9mm_P1.27mm" H 5200 2600 50  0001 C CNN
-F 3 "http://www.ti.com/lit/ds/symlink/tl081.pdf" H 5200 2600 50  0001 C CNN
+F 1 "LT6234CS8#PBF" H 5200 2876 50  0000 C CNN
+F 2 "Package_SO:SO-8_3.9x4.9mm_P1.27mm" H 5200 2600 50  0001 C CNN
+F 3 "https://www.analog.com/media/en/technical-documentation/data-sheets/623345fc.pdf" H 5200 2600 50  0001 C CNN
 	1    5200 2600
 	1    0    0    -1
@@
 Connection ~ 5500 2600
 $Comp
-L Amplifier_Operational:TL082 U1
-U 2 1 60F5B82B
+L Amplifier_Operational:LT6234 U1
+U 2 1 610B509A
 P 5950 4050
 F 0 "U1" H 5950 4417 50  0000 C CNN
-F 1 "TL082CDE4" H 5950 4326 50  0000 C CNN
-F 2 "Package_SO:SOIC-8_3.9x4.9mm_P1.27mm" H 5950 4050 50  0001 C CNN
-F 3 "http://www.ti.com/lit/ds/symlink/tl081.pdf" H 5950 4050 50  0001 C CNN
+F 1 "LT6234CS8#PBF" H 5950 4326 50  0000 C CNN
+F 2 "Package_SO:SO-8_3.9x4.9mm_P1.27mm" H 5950 4050 50  0001 C CNN
+F 3 "https://www.analog.com/media/en/technical-documentation/data-sheets/623345fc.pdf" H 5950 4050 50  0001 C CNN
 	2    5950 4050
 	1    0    0    -1
@@
 Connection ~ 5650 4150
 $Comp
-L Amplifier_Operational:TL082 U1
-U 3 1 60F654A5
+L Amplifier_Operational:LT6234 U1
+U 3 1 610BC20F
 P 9200 1450
 F 0 "U1" H 9158 1496 50  0000 L CNN
-F 1 "TL082CDE4" H 9158 1405 50  0000 L CNN
-F 2 "Package_SO:SOIC-8_3.9x4.9mm_P1.27mm" H 9200 1450 50  0001 C CNN
-F 3 "http://www.ti.com/lit/ds/symlink/tl081.pdf" H 9200 1450 50  0001 C CNN
+F 1 "LT6234CS8#PBF" H 9158 1405 50  0000 L CNN
+F 2 "Package_SO:SO-8_3.9x4.9mm_P1.27mm" H 9200 1450 50  0001 C CNN
+F 3 "https://www.analog.com/media/en/technical-documentation/data-sheets/623345fc.pdf" H 9200 1450 50  0001 C CNN
 	3    9200 1450
 	1    0    0    -1
 $EndComp
+$Comp
+L Device:C C10
+U 1 1 610AE00F
+P 5150 3100
+F 0 "C10" V 4898 3100 50  0000 C CNN
+F 1 "47pF" V 4989 3100 50  0000 C CNN
+F 2 "Capacitor_SMD:C_0201_0603Metric_Pad0.64x0.40mm_HandSolder" H 5188 2950 50  0001 C CNN
+F 3 "~" H 5150 3100 50  0001 C CNN
+	1    5150 3100
+	0    -1   -1   0
+$EndComp
+$Comp
+L Device:C C11
+U 1 1 610B8196
+P 5900 4550
+F 0 "C11" V 5648 4550 50  0000 C CNN
+F 1 "47pF" V 5739 4550 50  0000 C CNN
+F 2 "Capacitor_SMD:C_0201_0603Metric_Pad0.64x0.40mm_HandSolder" H 5938 4400 50  0001 C CNN
+F 3 "~" H 5900 4550 50  0001 C CNN
+	1    5900 4550
+	0    -1   -1   0
+$EndComp
+Wire Wire Line
+	5750 4550 5650 4550
+Connection ~ 5650 4550
+Wire Wire Line
+	5650 4550 5650 4800
+Wire Wire Line
+	6050 4550 6200 4550
+Connection ~ 6200 4550
+Wire Wire Line
+	6200 4550 6200 4300
+Wire Wire Line
+	5000 3100 4800 3100
+Connection ~ 4800 3100
+Wire Wire Line
+	4800 3100 4800 2700
+Wire Wire Line
+	5300 3100 5500 3100
+Connection ~ 5500 3100
+Wire Wire Line
+	5500 3100 5500 3400
 $EndSCHEMATC
